Commit message: Updated the position of the rplidar.

File: stacks/circles.urdf.xacro (robot description, xacro)
@@ -264,26 +264,27 @@
       </collision>
     </link>
-    <gazebo>
     <link name="rplidar_link">
-      <pose>0.08 0 0.42 0 0 0</pose>
       <visual name="visual">
-        <geometry>
-	  <cylinder>
-	    <radius>0.035</radius>
-	    <length>0.02</length>
-	  </cylinder>
+	<origin xyz="0 0 0" rpy="0 0 0"/>
+        <geometry>
+	  <cylinder length="0.02" radius="0.035"/>
         </geometry>
       </visual>
       <collision name="collision">
-        <geometry>
-	  <cylinder>
-	    <radius>0.035</radius>
-	    <length>0.02</length>
-	  </cylinder>
-        </geometry>
-      </collision>
-      <sensor name="rplidar" type="ray">
-        <ray>
-          <scan>
+	<origin xyz="0 0 0" rpy="0 0 0"/>
+	<geometry>
+	  <cylinder length="0.02" radius="0.035"/>
+        </geometry>
+      </collision>
+    </link>
+    <joint name="body_to_hokuyo" type="fixed">
+      <origin xyz="0.08 0.0  0.19310784" rpy="0 0 0"/>
+      <parent link="${parent}"/>
+      <child link="rplidar_link"/>
+    </joint>
+      <gazebo reference="rplidar_link">
+	<sensor name="rplidar" type="ray">
+	  <ray>
+	    <scan>
             <horizontal>
               <samples>360</samples>
@@ -312,22 +313,10 @@
           <alwaysOn>true</alwaysOn>
           <updateRate>6</updateRate>
-          <topicName>/scan_rplidar</topicName>
-          <frameName>/base_link</frameName>
+          <topicName>/rplidar_scan</topicName>
+          <frameName>/rplidar_link</frameName>
           <hokuyoMinIntensity>101</hokuyoMinIntensity>
         </plugin>
       </sensor>
-    </link>
-    <joint name="body_to_hokuyo" type="revolute">
-      <child>rplidar_link</child>
-      <parent>plate_3_link</parent>
-      <axis>
-        <xyz>0 0 0</xyz>
-        <limit>
-          <upper>0</upper>
-          <lower>0</lower>
-        </limit>
-      </axis>
-    </joint>
-  </gazebo>
+    </gazebo>
   </xacro:macro>
 </robot>

File: stacks/hexagons.urdf.xacro (robot description, xacro)
@@ -221,26 +221,27 @@
       </inertial>
     </link>
-    <gazebo>
     <link name="rplidar_link">
-      <pose>0.08 0 0.42 0 0 0</pose>
       <visual name="visual">
-        <geometry>
-	  <cylinder>
-	    <radius>0.035</radius>
-	    <length>0.02</length>
-	  </cylinder>
+	<origin xyz="0 0 0" rpy="0 0 0"/>
+        <geometry>
+	  <cylinder length="0.02" radius="0.035"/>
         </geometry>
       </visual>
       <collision name="collision">
-        <geometry>
-	  <cylinder>
-	    <radius>0.035</radius>
-	    <length>0.02</length>
-	  </cylinder>
-        </geometry>
-      </collision>
-      <sensor name="rplidar" type="ray">
-        <ray>
-          <scan>
+	<origin xyz="0 0 0" rpy="0 0 0"/>
+	<geometry>
+	  <cylinder length="0.02" radius="0.035"/>
+        </geometry>
+      </collision>
+    </link>
+    <joint name="body_to_hokuyo" type="fixed">
+      <origin xyz="0.08 0.0  0.1974" rpy="0 0 0"/>
+      <parent link="${parent}"/>
+      <child link="rplidar_link"/>
+    </joint>
+      <gazebo reference="rplidar_link">
+	<sensor name="rplidar" type="ray">
+	  <ray>
+	    <scan>
             <horizontal>
               <samples>360</samples>
@@ -269,22 +270,10 @@
           <alwaysOn>true</alwaysOn>
           <updateRate>6</updateRate>
-          <topicName>/scan_rplidar</topicName>
-          <frameName>/base_link</frameName>
+          <topicName>/rplidar_scan</topicName>
+          <frameName>/rplidar_link</frameName>
           <hokuyoMinIntensity>101</hokuyoMinIntensity>
         </plugin>
       </sensor>
-    </link>
-    <joint name="body_to_hokuyo" type="revolute">
-      <child>rplidar_link</child>
-      <parent>plate_top_link</parent>
-      <axis>
-        <xyz>0 0 0</xyz>
-        <limit>
-          <upper>0</upper>
-          <lower>0</lower>
-        </limit>
-      </axis>
-    </joint>
-  </gazebo>
+    </gazebo>
   </xacro:macro>
 </robot>
