Commit message: Updated models from stl to dae

File: turtlebot_description/urdf/sensors/realsense.urdf.xacro (robot description, xacro)
@@ -16,5 +16,5 @@
        <origin xyz="0 0 0" rpy="0 0 0"/>
         <geometry>
-         <mesh filename="package://turtlebot_description/meshes/sensors/realsense.stl"/>
+         <mesh filename="package://turtlebot_description/meshes/sensors/realsense.dae"/>
         </geometry>
       </visual>

File: turtlebot_description/urdf/stand.urdf.xacro (robot description, xacro)
@@ -5,5 +5,5 @@
       <visual>
 	<geometry>
-	  <mesh filename="file://$(find turtlebot_description)/meshes/stand/base.stl"></mesh>
+	  <mesh filename="file://$(find turtlebot_description)/meshes/stand/base.dae"></mesh>
 	</geometry>
       </visual>
@@ -12,5 +12,5 @@
       <visual>
 	<geometry>
-	  <mesh filename="file://$(find turtlebot_description)/meshes/stand/fork.stl"></mesh>
+	  <mesh filename="file://$(find turtlebot_description)/meshes/stand/fork.dae"></mesh>
 	</geometry>
       </visual>
@@ -19,5 +19,5 @@
       <visual>
 	<geometry>
-	  <mesh filename="file://$(find turtlebot_description)/meshes/stand/plate.stl"></mesh>
+	  <mesh filename="file://$(find turtlebot_description)/meshes/stand/plate.dae"></mesh>
 	</geometry>
       </visual>
@@ -26,5 +26,5 @@
       <visual>
 	<geometry>
-	  <mesh filename="file://$(find turtlebot_description)/meshes/stand/screen.stl"></mesh>
+	  <mesh filename="file://$(find turtlebot_description)/meshes/stand/screen.dae"></mesh>
 	</geometry>
       </visual>
