Commit message: Added an option to rotate camera stand elements

File: turtlebot_description/urdf/stand.urdf.xacro (robot description, xacro)
@@ -8,4 +8,9 @@
 	</geometry>
       </visual>
+      <inertial>
+	<origin xyz="0 0 0" rpy="0 0 0"/>
+	<mass value="0.01"/>
+	<inertia ixx="0.001" ixy="0.0" ixz="0.0" iyy="0.001" iyz="0.0" izz="0.001"/>
+      </inertial>
     </link>
     <link name="realsense_fork_stand">
@@ -15,4 +20,9 @@
 	</geometry>
       </visual>
+      <inertial>
+	<origin xyz="0 0 0" rpy="0 0 0"/>
+	<mass value="0.01"/>
+	<inertia ixx="0.001" ixy="0.0" ixz="0.0" iyy="0.001" iyz="0.0" izz="0.001"/>
+      </inertial>
     </link>
     <link name="realsense_plate_stand">
@@ -22,4 +32,9 @@
 	</geometry>
       </visual>
+      <inertial>
+	<origin xyz="0 0 0" rpy="0 0 0"/>
+	<mass value="0.01"/>
+	<inertia ixx="0.001" ixy="0.0" ixz="0.0" iyy="0.001" iyz="0.0" izz="0.001"/>
+      </inertial>
     </link>
     <link name="realsense_screen_stand">
@@ -29,4 +44,9 @@
 	</geometry>
       </visual>
+      <inertial>
+	<origin xyz="0 0 0" rpy="0 0 0"/>
+	<mass value="0.01"/>
+	<inertia ixx="0.001" ixy="0.0" ixz="0.0" iyy="0.001" iyz="0.0" izz="0.001"/>
+      </inertial>
     </link>
     <joint name="parent_base_joint" type="fixed">
@@ -36,22 +56,46 @@
       <axis xyz="0 1 0" />
     </joint>
-    <joint name="base_fork_joint" type="fixed">
+    <joint name="base_fork_joint" type="continuous">
       <parent link="realsense_base_stand"/>
       <child link="realsense_fork_stand"/>
       <origin xyz="0 0 0" rpy="0 0 0"/>
-      <axis xyz="0 1 0" />
+      <axis xyz="0 0 1" />
+      <limit effort="750000.0" velocity="30.0"/>
     </joint>
-    <joint name="fork_plate_joint" type="fixed">
+    <joint name="fork_plate_joint" type="continuous">
       <parent link="realsense_fork_stand"/>
       <child link="realsense_plate_stand"/>
-      <origin xyz="0 0 0" rpy="0 0 0"/>
+      <origin xyz="0 0 0.197" rpy="0 0 0"/>
       <axis xyz="0 1 0" />
+      <limit effort="750000.0" velocity="30.0"/>
     </joint>
     <joint name="plate_screen_joint" type="fixed">
       <parent link="realsense_plate_stand"/>
       <child link="realsense_screen_stand"/>
-      <origin xyz="0 0 0" rpy="0 0 0"/>
+      <origin xyz="0 0 -0.197" rpy="0 0 0"/>
       <axis xyz="0 1 0" />
     </joint>
+    <transmission name="base_fork_joint_transmission">
+	<type>transmission_interface/SimpleTransmission</type>
+	<joint name="base_fork_joint">
+	    <hardwareInterface>VelocityJointInterface</hardwareInterface>
+	    <mechanicalReduction>1</mechanicalReduction>
+	</joint>
+	<actuator name="base_fork_joint_actuator">
+	    <hardwareInterface>VelocityJointInterface</hardwareInterface>
+	    <mechanicalReduction>1</mechanicalReduction>
+	</actuator>
+    </transmission>
+    <transmission name="fork_plate_joint_transmission">
+	<type>transmission_interface/SimpleTransmission</type>
+	<joint name="fork_plate_joint">
+	    <hardwareInterface>VelocityJointInterface</hardwareInterface>
+	    <mechanicalReduction>1</mechanicalReduction>
+	</joint>
+	<actuator name="fork_plate_joint_actuator">
+	    <hardwareInterface>VelocityJointInterface</hardwareInterface>
+	    <mechanicalReduction>1</mechanicalReduction>
+	</actuator>
+    </transmission>
     <gazebo reference="realsense_base_stand">
       <material>Gazebo/Grey</material>
@@ -66,4 +110,7 @@
       <material>Gazebo/Grey</material>
     </gazebo>
+    <gazebo>
+    <plugin name="gazebo_ros_control" filename="libgazebo_ros_control.so"/>
+    </gazebo>
   </xacro:macro>
 </robot>
