Commit message: Add a screen into the model

File: turtlebot_description/robots/kobuki_hexagons_realsense.urdf.xacro (robot description, xacro)
@@ -7,8 +7,7 @@
 <robot name="turtlebot" xmlns:xacro="http://ros.org/wiki/xacro">
   <xacro:include filename="$(find turtlebot_description)/urdf/turtlebot_library.urdf.xacro" />
-  <xacro:include filename="$(find turtlebot_description)/urdf/stand.urdf.xacro" />
   <kobuki/>
   <stack_hexagons parent="base_link"/>
   <sensor_realsense_stand parent="base_link" x="0" y="0" z="0.4" roll="0" pitch="0" yaw="0"/>
-  <sensor_realsense  parent="realsense_plate_stand"/>
+  <sensor_realsense  parent="realsense_screen_stand"/>
 </robot>

File: turtlebot_description/urdf/sensors/realsense.urdf.xacro (robot description, xacro)
@@ -29,5 +29,5 @@
       <parent link="camera_link"/>
       <child link="camera_base"/>
-      <origin xyz="0.025 0 0.2" rpy="0 0 0"/>
+      <origin xyz="0.025 0 0.37" rpy="0 0 0"/>
       <axis xyz="0 1 0" />
     </joint>

File: turtlebot_description/urdf/stand.urdf.xacro (robot description, xacro)
@@ -23,4 +23,11 @@
       </visual>
     </link>
+    <link name="realsense_screen_stand">
+      <visual>
+	<geometry>
+	  <mesh filename="file://$(find turtlebot_description)/meshes/stand/screen.stl"></mesh>
+	</geometry>
+      </visual>
+    </link>
     <joint name="parent_base_joint" type="fixed">
       <parent link="${parent}"/>
@@ -41,4 +48,10 @@
       <axis xyz="0 1 0" />
     </joint>
+    <joint name="plate_screen_joint" type="fixed">
+      <parent link="realsense_plate_stand"/>
+      <child link="realsense_screen_stand"/>
+      <origin xyz="0 0 0" rpy="0 0 0"/>
+      <axis xyz="0 1 0" />
+    </joint>
     <gazebo reference="realsense_base_stand">
       <material>Gazebo/Grey</material>
@@ -50,4 +63,7 @@
       <material>Gazebo/Grey</material>
     </gazebo>
+    <gazebo reference="realsense_screen_stand">
+      <material>Gazebo/Grey</material>
+    </gazebo>
   </xacro:macro>
 </robot>

File: turtlebot_description/urdf/turtlebot_library.urdf.xacro (robot description, xacro)
@@ -13,4 +13,6 @@
   <xacro:include filename="$(find turtlebot_description)/urdf/stacks/circles.urdf.xacro"/>
   <xacro:include filename="$(find turtlebot_description)/urdf/stacks/hexagons.urdf.xacro"/>
+  <!-- Stand for realsense -->
+  <xacro:include filename="$(find turtlebot_description)/urdf/stand.urdf.xacro" />
   <!-- 3D Sensors -->
   <xacro:include filename="$(find turtlebot_description)/urdf/sensors/kinect.urdf.xacro"/>

Commit message: Added spacer for camera

File: turtlebot_description/robots/kobuki_hexagons_realsense.urdf.xacro (robot description, xacro)
@@ -9,5 +9,5 @@
   <kobuki/>
   <stack_hexagons parent="base_link"/>
-  <sensor_realsense_stand parent="base_link" x="0" y="0" z="0.4" roll="0" pitch="0" yaw="0"/>
+  <sensor_realsense_stand parent="base_link" x="0" y="0" z="0.425" roll="0" pitch="0" yaw="0"/>
   <sensor_realsense  parent="realsense_screen_stand"/>
 </robot>

File: turtlebot_description/urdf/stand.urdf.xacro (robot description, xacro)
@@ -2,4 +2,16 @@
 <robot name="realsense_stand" xmlns:xacro="http://ros.org/wiki/xacro">
   <xacro:macro name="sensor_realsense_stand" params="parent x y z roll pitch yaw">
+    <link name="realsense_base_spacer">
+      <visual>
+	<geometry>
+	  <cylinder length="0.05" radius="0.05"/>
+	</geometry>
+      </visual>
+      <inertial>
+	<origin xyz="0 0 0" rpy="0 0 0"/>
+	<mass value="0.01"/>
+	<inertia ixx="0.001" ixy="0.0" ixz="0.0" iyy="0.001" iyz="0.0" izz="0.001"/>
+      </inertial>
+    </link>
     <link name="realsense_base_stand">
       <visual>
@@ -50,8 +62,14 @@
       </inertial>
     </link>
-    <joint name="parent_base_joint" type="fixed">
+    <joint name="parent_base_spacer_joint" type="fixed">
       <parent link="${parent}"/>
+      <child link="realsense_base_spacer"/>
+      <origin xyz="${x} ${y} ${z}" rpy="${roll} ${pitch} ${yaw}"/>
+      <axis xyz="0 1 0" />
+    </joint>
+    <joint name="base_socaer_base_joint" type="fixed">
+      <parent link="realsense_base_spacer"/>
       <child link="realsense_base_stand"/>
-      <origin xyz="${x} ${y} ${z}" rpy="${roll} ${pitch} ${yaw}"/>
+      <origin xyz="0 0 0.025" rpy="0 0 0"/>
       <axis xyz="0 1 0" />
     </joint>

Commit message: Updated the position of the lidar, added laptop

File: turtlebot_description/robots/kobuki_hexagons_realsense.urdf.xacro (robot description, xacro)
@@ -9,5 +9,5 @@
   <kobuki/>
   <stack_hexagons parent="base_link"/>
-  <sensor_realsense_stand parent="base_link" x="0" y="0" z="0.425" roll="0" pitch="0" yaw="0"/>
+  <sensor_realsense_stand parent="base_link" x="0" y="0" z="0.418" roll="0" pitch="0" yaw="0"/>
   <sensor_realsense  parent="realsense_screen_stand"/>
 </robot>

File: turtlebot_description/urdf/stacks/hexagons.urdf.xacro (robot description, xacro)
@@ -128,8 +128,8 @@
   <xacro:macro name="stack_hexagons" params="parent">
     <stack_bottom_pole parent="${parent}" number="0" x_loc= "0.120" y_loc= "0.082" z_loc="0.1028"/>
-    <stack_bottom_pole parent="${parent}" number="1" x_loc= "0.055" y_loc= "0.120" z_loc="0.1028"/>
+<!--     <stack_bottom_pole parent="${parent}" number="1" x_loc= "0.055" y_loc= "0.120" z_loc="0.1028"/> -->
     <stack_bottom_pole parent="${parent}" number="2" x_loc="-0.055" y_loc= "0.120" z_loc="0.1028"/>
     <stack_bottom_pole parent="${parent}" number="3" x_loc= "0.120" y_loc="-0.082" z_loc="0.1028"/>
-    <stack_bottom_pole parent="${parent}" number="4" x_loc= "0.055" y_loc="-0.120" z_loc="0.1028"/>
+<!--     <stack_bottom_pole parent="${parent}" number="4" x_loc= "0.055" y_loc="-0.120" z_loc="0.1028"/> -->
     <stack_bottom_pole parent="${parent}" number="5" x_loc="-0.055" y_loc="-0.120" z_loc="0.1028"/>
     <joint name="plate_bottom_joint" type="fixed">
@@ -159,5 +159,5 @@
       </inertial>
     </link>
-    <joint name="plate_middle_joint" type="fixed">
+<!--    <joint name="plate_middle_joint" type="fixed">
       <origin xyz="-0.01364 0.0 0.34" rpy="0 0 0"/>
       <parent link="${parent}"/>
@@ -184,17 +184,17 @@
                  izz="0.006656" />
       </inertial>
-    </link>
+    </link>-->
     <stack_top_pole parent="${parent}" number="0" x_loc= "0.0381" y_loc= "0.1505" z_loc="0.235"/>
     <stack_top_pole parent="${parent}" number="1" x_loc= "0.0381" y_loc="-0.1505" z_loc="0.235"/>
     <stack_top_pole parent="${parent}" number="2" x_loc="-0.0381" y_loc= "0.1505" z_loc="0.235"/>
     <stack_top_pole parent="${parent}" number="3" x_loc="-0.0381" y_loc="-0.1505" z_loc="0.235"/>
-    <stack_middle_pole parent="${parent}" number="0" x_loc= "0.0381" y_loc= "0.1505" z_loc="0.363"/>
-    <stack_middle_pole parent="${parent}" number="1" x_loc= "0.0381" y_loc="-0.1505" z_loc="0.363"/>
-    <stack_middle_pole parent="${parent}" number="2" x_loc="-0.0381" y_loc= "0.1505" z_loc="0.363"/>
-    <stack_middle_pole parent="${parent}" number="3" x_loc="-0.0381" y_loc="-0.1505" z_loc="0.363"/>
+    <stack_middle_pole parent="${parent}" number="0" x_loc= "0.0381" y_loc= "0.1505" z_loc="0.356"/>
+    <stack_middle_pole parent="${parent}" number="1" x_loc= "0.0381" y_loc="-0.1505" z_loc="0.356"/>
+    <stack_middle_pole parent="${parent}" number="2" x_loc="-0.0381" y_loc= "0.1505" z_loc="0.356"/>
+    <stack_middle_pole parent="${parent}" number="3" x_loc="-0.0381" y_loc="-0.1505" z_loc="0.356"/>
 <!--    <stack_3d_sensor_pole parent="${parent}" number="0" x_loc="-0.12" y_loc= "-0.015" z_loc="0.29"/>
     <stack_3d_sensor_pole parent="${parent}" number="1" x_loc="-0.12" y_loc="0.015" z_loc="0.29"/>-->
     <joint name="plate_top_joint" type="fixed">
-      <origin xyz="-0.01364 0.0  0.3966" rpy="0 0 0"/>
+      <origin xyz="-0.01364 0.0  0.3896" rpy="0 0 0"/>
       <parent link="${parent}"/>
       <child link="plate_top_link"/>
@@ -221,4 +221,17 @@
       </inertial>
     </link>
+    <link name="laptop_link">
+      <visual name="visual">
+	<origin xyz="0 0 0" rpy="0 0 0"/>
+        <geometry>
+	  <mesh filename="package://turtlebot_description/meshes/laptop/laptop.dae" scale="0.73 0.73 0.73"/>
+        </geometry>
+      </visual>
+    </link>
+    <joint name="laptop_to_parent" type="fixed">
+      <origin xyz="0 0.0 0.13" rpy="0 0 0"/>
+      <parent link="${parent}"/>
+      <child link="laptop_link"/>
+    </joint>
     <link name="rplidar_link">
       <visual name="visual">
@@ -236,5 +249,5 @@
     </link>
     <joint name="body_to_hokuyo" type="fixed">
-      <origin xyz="-0.12 0.0  0.29" rpy="0 3.1415 0"/>
+      <origin xyz="0.05 0.0 0.12" rpy="0 0 0"/>
       <parent link="${parent}"/>
       <child link="rplidar_link"/>
